File: hardware/pokeboy-hw/pokeboy-hw.kicad_pcb (KiCad board)
At the start: 4 copper layers, 79.4 x 119.4 mm, 110 parts, among them J1 USB Micro-B data/power, J2 LiPo 1S + / NTC / -, J3 POWER SWITCH PADS, J4 8 OHM SPEAKER PADS, J5 EA TFT020-23AINN RGB666, J6 UART TEST PADS, J7 RECOVERY SHORT PADS, J8 RESET SHORT PADS, J9 104031-0811, SW1 EVQ-P1905M, SW2 EVQ-P1905M, SW3 EVQ-P1905M, SW4 EVQ-P1905M, SW5 B3AL-1001P, SW6 B3AL-1001P, SW7 EVQ-P2B02B, SW8 EVQ-P2B02B, U1 OSD3358-1G-ISM, U2 BQ24074RGT, U3 TPS63802DLAR, U4 TPS62162DSG, U5 TPS61165DRV, U6 MAX98357AETE+T, U7 TPD2EUSB30, Y1 24 MHz

Commit message: hw: reconcile the schematic to the board and clean up the CPL
The schematic did not describe this board. It still held the Luckfox
Core1106 (Rockchip RV1106, 112 numeric pins) as U1 while the board is an
Octavo OSD3358 BGA-256; 17 parts existed only in the PCB; 6 existed only
in the schematic; and ERC therefore only ever covered 99 of 110 parts.

Schematic, matching the sheet's existing style (labels on pins, no wires):

- Replace U1 with an OSD3358_BGA256 symbol whose 132 pins are the ball
  designators the board uses. GENERATED FROM THE LAYOUT - it makes the two
  files agree, it does not verify the ball map against Octavo's datasheet.
- Add the 17 PCB-only parts: Y1, J9, RN7-RN10, R102, R104-R109, C102,
  C103, C105, C106. New symbols for the crystal, an 11-way connector and
  a real MAX98357A (U6 was a PAM8302AAD, 8 pins, MSOP-8).
- Drop the obsolete analog line-in path C17/C18/C19/R24/R25 - the board
  has no CODEC_LINEOUT/LINE_FILT/AMP_IN nets, U6 is I2S.
- Correct C20/C21: schematic had them on AUX_3V3, the board has them on
  SYS_5V beside U6, whose VDD is SYS_5V.
- Remove 45 no-connects left dangling by the U1 swap; snap new placement
  to the 1.27 mm grid.

Board:

- Add R26, the 100k AMP_EN pull-down, at (17.5,36.0). It was schematic-
  only, so the amp enable had no pull-down; it also consumes a dangling
  AMP_EN stub.
- Mark R9/R19 DNP and exclude J2-J8 from pos files. DNP previously lived
  only in the hand-written BOM, so the CPL told the assembler to fit
  parts the BOM says not to fit. CPL drops 109 -> 101 placeable rows.
- Library-qualify all 18 unqualified footprint ids, register
  Connector_Card, and export the crystal footprint to Pokeboy.pretty.

Verification: schematic netlist and PCB connectivity are now identical -
0 nets differing in membership, none present on only one side. DRC 0
errors / 0 unconnected / 80 warnings (was 99). ERC 5, down from 87 once
it began covering all 110 parts.

Two real defects found and NOT fixed, both needing the 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
Parts:
- added R26: 100k, Resistor_SMD:R_0402_1005Metric, F.Cu at (17.5, 36.0)
- C102, C103, C105: footprint C_0402_1005Metric -> Capacitor_SMD:C_0402_1005Metric
- C106: footprint C_0805_2012Metric -> Capacitor_SMD:C_0805_2012Metric
- J9: footprint microSD_HC_Molex_104031-0811 -> Connector_Card:microSD_HC_Molex_104031-0811
- R102, R104, R105, R106, R107, R108, R109: footprint R_0402_1005Metric -> Resistor_SMD:R_0402_1005Metric
- RN10, RN7, RN8, RN9: footprint R_Array_Convex_4x0603 -> Resistor_SMD:R_Array_Convex_4x0603
- U6: footprint TQFN-16-1EP_3x3mm_P0.5mm_EP1.23x1.23mm -> Package_DFN_QFN:TQFN-16-1EP_3x3mm_P0.5mm_EP1.23x1.23mm
- Y1: footprint PocketBeagle.pretty:CRYSTAL_5X3.2MM -> Pokeboy:CRYSTAL_5X3.2MM
Changed lines of the file:
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@@
 		(sheetname "/")
 		(sheetfile "pokeboy-hw.kicad_sch")
-		(attr smd)
+		(attr smd exclude_from_pos_files)
 		(fp_line
 			(start -3.5 -1.5)
@@
 		)
 	)
-	(footprint "C_0402_1005Metric"
+	(footprint "Capacitor_SMD:C_0402_1005Metric"
 		(layer "F.Cu")
 		(at 27 34.5)
@@
 		)
 	)
-	(footprint "R_0402_1005Metric"
+	(footprint "Resistor_SMD:R_0402_1005Metric"
 		(layer "F.Cu")
 		(at 46.6 33.8)
@@
 		)
 	)
-	(footprint "TQFN-16-1EP_3x3mm_P0.5mm_EP1.23x1.23mm"
+	(footprint "Package_DFN_QFN:TQFN-16-1EP_3x3mm_P0.5mm_EP1.23x1.23mm"
 		(layer "F.Cu")
 		(at 12 43.5)
@@
 		)
 	)
-	(footprint "microSD_HC_Molex_104031-0811"
+	(footprint "Connector_Card:microSD_HC_Molex_104031-0811"
 		(layer "F.Cu")
 		(at 57 46 90)
@@
 		)
 	)
-	(footprint "R_0402_1005Metric"
+	(footprint "Resistor_SMD:R_0402_1005Metric"
 		(layer "F.Cu")
 		(at 46.6 37.2)
@@
 		)
 	)
-	(footprint "R_0402_1005Metric"
+	(footprint "Resistor_SMD:R_0402_1005Metric"
 		(layer "F.Cu")
 		(at 15.316 15.65)
@@
 		)
 	)
-	(footprint "R_Array_Convex_4x0603"
+	(footprint "Resistor_SMD:R_Array_Convex_4x0603"
 		(layer "F.Cu")
 		(at 39.3 26.5 90)
@@
 		)
 	)
-	(footprint "R_0402_1005Metric"
+	(footprint "Resistor_SMD:R_0402_1005Metric"
 		(layer "F.Cu")
 		(at 49 33.8)
@@
 		(sheetname "/")
 		(sheetfile "pokeboy-hw.kicad_sch")
-		(attr smd)
+		(attr smd exclude_from_pos_files)
 		(fp_line
 			(start -6.5 -1.25)
@@
 		(sheetname "/")
 		(sheetfile "pokeboy-hw.kicad_sch")
-		(attr smd)
+		(attr smd exclude_from_pos_files dnp)
 		(fp_line
 			(start -0.153641 -0.38)
@@
 		(sheetname "/")
 		(sheetfile "pokeboy-hw.kicad_sch")
-		(attr smd)
+		(attr smd exclude_from_pos_files)
 		(fp_line
 			(start -1.5 -1)
@@
 	(footprint "Resistor_SMD:R_0402_1005Metric"
 		(layer "F.Cu")
+		(at 17.5 36 90)
+		(descr "Resistor SMD 0402 (1005 Metric), square (rectangular) end terminal, IPC-7351 nominal, (Body size source: IPC-SM-782 page 72, https://www.pcb-3d.com/wordpress/wp-content/uploads/ipc-sm-782a_amendment_1_and_2.pdf), generated with kicad-footprint-generator")
+		(tags "resistor")
+		(property "Reference" "R26"
+			(at 0 -1.17 90)
+			(layer "F.SilkS")
+			(hide yes)
+			(effects
+				(font
+					(size 1 1)
+					(thickness 0.15)
+				)
+			)
+		)
+		(property "Value" "100k"
+			(at 0 1.17 90)
+			(layer "F.Fab")
+			(hide yes)
+			(effects
+				(font
+					(size 1 1)
+					(thickness 0.15)
+				)
+			)
+		)
+		(property "Datasheet" ""
+			(at 0 0 90)
+			(layer "F.Fab")
+			(hide yes)
+			(effects
+				(font
+					(size 1.27 1.27)
+					(thickness 0.15)
+				)
+			)
+		)
+		(property "Description" ""
+			(at 0 0 90)
+			(layer "F.Fab")
+			(hide yes)
+			(effects
+				(font
+					(size 1.27 1.27)
+					(thickness 0.15)
+				)
+			)
+		)
+		(attr smd)
+		(fp_line
+			(start -0.153641 -0.38)
+			(end 0.153641 -0.38)
+			(stroke
+				(width 0.12)
+				(type solid)
+			)
+			(layer "F.SilkS")
+		)
+		(fp_line
+			(start -0.153641 0.38)
+			(end 0.153641 0.38)
+			(stroke
+				(width 0.12)
+				(type solid)
+			)
+			(layer "F.SilkS")
+		)
+		(fp_rect
+			(start -0.93 -0.47)
+			(end 0.93 0.47)
+			(stroke
+				(width 0.05)
+				(type solid)
+			)
+			(fill no)
+			(layer "F.CrtYd")
+		)
+		(fp_rect
+			(start -0.525 -0.27)
+			(end 0.525 0.27)
+			(stroke
+				(width 0.1)
+				(type solid)
+			)
+			(fill no)
+			(layer "F.Fab")
+		)
+		(fp_text user "${REFERENCE}"
+			(at 0 0 90)
+			(layer "F.Fab")
+			(effects
+				(font
+					(size 0.26 0.26)
+					(thickness 0.04)
+				)
+			)
+		)
+		(pad "1" smd roundrect
+			(at -0.51 0 90)
+			(size 0.54 0.64)
+			(layers "F.Cu" "F.Mask" "F.Paste")
+			(roundrect_rratio 0.25)
+			(net 3 "/AMP_EN")
+		)
+		(pad "2" smd roundrect
+			(at 0.51 0 90)
+			(size 0.54 0.64)
+			(layers "F.Cu" "F.Mask" "F.Paste")
+			(roundrect_rratio 0.25)
+			(net 1 "/GND")
+		)
+		(embedded_fonts no)
+		(model "${KICAD9_3DMODEL_DIR}/Resistor_SMD.3dshapes/R_0402_1005Metric.step"
+			(offset
+				(xyz 0 0 0)
+			)
+			(scale
+				(xyz 1 1 1)
+			)
+			(rotate
+				(xyz 0 0 0)
+			)
+		)
+	)
+	(footprint "Resistor_SMD:R_0402_1005Metric"
+		(layer "F.Cu")
 		(at 73.5 13.2 90)
 		(descr "Resistor SMD 0402 (1005 Metric), square (rectangular) end terminal, IPC-7351 nominal, (Body size source: IPC-SM-782 page 72, https://www.pcb-3d.com/wordpress/wp-content/uploads/ipc-sm-782a_amendment_1_and_2.pdf), generated with kicad-footprint-generator")
@@
 		)
 	)
-	(footprint "R_0402_1005Metric"
+	(footprint "Resistor_SMD:R_0402_1005Metric"
 		(layer "F.Cu")
 		(at 49 35.5)
@@
 		)
 	)
-	(footprint "PocketBeagle.pretty:CRYSTAL_5X3.2MM"
+	(footprint "Pokeboy:CRYSTAL_5X3.2MM"
 		(layer "F.Cu")
 		(at 12.522 15.65 90)
@@
 		)
 	)
-	(footprint "R_Array_Convex_4x0603"
+	(footprint "Resistor_SMD:R_Array_Convex_4x0603"
 		(layer "F.Cu")
 		(at 39.3 14.5 90)
@@
 		(sheetname "/")
 		(sheetfile "pokeboy-hw.kicad_sch")
-		(attr smd)
+		(attr smd exclude_from_pos_files)
 		(fp_line
 			(start -2.5 -1.6)
@@
 		(embedded_fonts no)
 	)
-	(footprint "R_Array_Convex_4x0603"
+	(footprint "Resistor_SMD:R_Array_Convex_4x0603"
 		(layer "F.Cu")
 		(at 39.3 18.5 90)
@@
 		)
 	)
-	(footprint "C_0402_1005Metric"
+	(footprint "Capacitor_SMD:C_0402_1005Metric"
 		(layer "F.Cu")
 		(at 15.316 13.999)
@@
 		(sheetname "/")
 		(sheetfile "pokeboy-hw.kicad_sch")
-		(attr smd)
+		(attr smd exclude_from_pos_files dnp)
 		(fp_line
 			(start -0.153641 -0.38)
@@
 		(sheetname "/")
 		(sheetfile "pokeboy-hw.kicad_sch")
-		(attr smd)
+		(attr smd exclude_from_pos_files)
 		(fp_line
 			(start -2.405 -1)
@@
 		)
 	)
-	(footprint "R_0402_1005Metric"
+	(footprint "Resistor_SMD:R_0402_1005Metric"
 		(layer "F.Cu")
 		(at 46.6 35.5)
@@
 		(sheetname "/")
 		(sheetfile "pokeboy-hw.kicad_sch")
-		(attr smd)
+		(attr smd exclude_from_pos_files)
 		(fp_line
 			(start -1.5 -1)
@@
 		)
 	)
-	(footprint "C_0805_2012Metric"
+	(footprint "Capacitor_SMD:C_0805_2012Metric"
 		(layer "F.Cu")
 		(at 31 34.5)
@@
 		)
 	)
-	(footprint "R_Array_Convex_4x0603"
+	(footprint "Resistor_SMD:R_Array_Convex_4x0603"
 		(layer "F.Cu")
 		(at 39.3 22.5 90)
@@
 		)
 	)
-	(footprint "R_0402_1005Metric"
+	(footprint "Resistor_SMD:R_0402_1005Metric"
 		(layer "F.Cu")
 		(at 49 37.2)
@@
 		(sheetname "/")
 		(sheetfile "pokeboy-hw.kicad_sch")
-		(attr smd)
+		(attr smd exclude_from_pos_files)
 		(fp_line
 			(start -2.5 -1.5)
@@
 		(embedded_fonts no)
 	)
-	(footprint "C_0402_1005Metric"
+	(footprint "Capacitor_SMD:C_0402_1005Metric"
 		(layer "F.Cu")
 		(at 15.316 17.301)
@@
 		(width 0.15)
 		(layer "F.Cu")
+		(net 3)
+	)
+	(segment
+		(start 17.5 36.51)
+		(end 17.5 37)
+		(width 0.15)
+		(layer "F.Cu")

Commit message: hw: verify U1's ball map against Octavo and tie the balls it requires
The OSD3358 symbol was generated from the layout, so it could only prove the
schematic and the board agreed - not that either was right. Checking it against
Octavo's own PocketBeagle reference design (OSD3358-512M-BSM, identical BGA-256
ball map) confirms every peripheral assignment: LCD, MMC0, I2C0, UART0, MCASP0,
USB0 and OSC0 all land on balls whose documented signal names match. Pin names
in the symbol now come from that library, so the sheet shows the datasheet
signal beside the net and any future divergence is visible.

The same check found balls the reference ties that this board left floating:

- N10/N11 PMIC_POWER_EN <-> PMIC_PWR_EN. This gates the PMIC's enable, so as it
  stood the SiP would not have powered up at all.
- N4/N5 PMIC_LDO_PGOOD <-> RTC_PWRONRSTN.
- N12/P11 PMIC_PGOOD -> PWRONRSTN, which releases reset.
- A7/B7 SYS_ADC_1P8V -> VREFP and A9/B9 AGND_ADC -> VREFN. AIN0 is in use for
  BAT_SENSE, and without a reference pair that reading is meaningless.

All five are adjacent-ball ties inside the 1.27 mm field, routed on F.Cu.

The two stranded Core1106 rails are also retired:

- CORE_3V3 fed R12/R13/R18/R32 from nothing. Its pull-ups all bias nets in the
  VDDSHV I/O domain, so it is merged onto OSD_3V3A, which supplies that domain.
  SD_CLK walls off F.Cu at x=50.772 and the SD fanout fills In1 and In2 in the
  gap, so no new via fits; both sides already own a through via and B.Cu between
  them is clear, so the join is one bottom-layer track and no new via.
- The In1 spine and F.Cu stub that carried CORE_3V3 west to the old module's
  landing pads are removed - R12/R13/R18 reach the net over In2 and R32 on F.Cu.
- CORE_1V8 reached only TP1. All eight SYS_VDD_1P8V balls sit in the interior of
  the field ringed by DGND, and Octavo's own PocketBeagle leaves VDD_1V8 with no
  external connection either, so the rail cannot be brought out. TP1 is removed
  rather than left wired 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
Parts:
- removed TP1: CORE 1V8 TEST, TestPoint:TestPoint_Pad_D1.0mm
Connections:
- J9 pad 11: (no net) -> /GND
- R12 pad 1: /CORE_3V3 -> /OSD_3V3A
- R13 pad 1: /CORE_3V3 -> /OSD_3V3A
- R18 pad 1: /CORE_3V3 -> /OSD_3V3A
- R32 pad 1: /CORE_3V3 -> /OSD_3V3A
- U1 pad A7: (no net) -> /ADC_VREFP
- U1 pad A9: (no net) -> /ADC_VREFN
- U1 pad B7: (no net) -> /ADC_VREFP
- U1 pad B9: (no net) -> /ADC_VREFN
- U1 pad N10: (no net) -> /PMIC_PWR_EN
- U1 pad N11: (no net) -> /PMIC_PWR_EN
- U1 pad N12: (no net) -> /PMIC_PGOOD
- U1 pad N4: (no net) -> /RTC_PWRONRSTN
- U1 pad N5: (no net) -> /RTC_PWRONRSTN
- U1 pad P11: (no net) -> /PMIC_PGOOD
- U6 pad 12: (no net) -> unconnected-(U6-NC-Pad12)
- U6 pad 13: (no net) -> unconnected-(U6-NC-Pad13)
- U6 pad 5: (no net) -> unconnected-(U6-NC-Pad5)
- U6 pad 6: (no net) -> unconnected-(U6-NC-Pad6)
Routing:
- net /CORE_3V3: track 88.7 -> 0.00 mm, vias 4 -> 0
- net /OSD_3V3A: track 74.9 -> 144.2 mm, vias 4 -> 7
- net /CORE_1V8: track 30.2 -> 0.00 mm
- net /PMIC_PGOOD: track 0.00 -> 1.80 mm
- net /RTC_PWRONRSTN: track 0.00 -> 1.27 mm
- net /PMIC_PWR_EN: track 0.00 -> 1.27 mm
- net /ADC_VREFP: track 0.00 -> 1.27 mm
- net /ADC_VREFN: track 0.00 -> 1.27 mm
Other:
- board text added: "0.8 mm 4-LAYER - REV PROTO-B"
- board text added: "OSD3358"
- board text added: "POKEBOY OSD3358 / RGB666 / 1S LIPO"
- board text removed: "0.8 mm 4-LAYER - REV PROTO-A"
- board text removed: "CORE1106"
- board text removed: "POKEBOY CORE1106 / RGB666 / 1S LIPO"

Commit message: hw: remove dead copper - 34 dangling stubs, orphan via, isolated pour islands
DRC warning triage (78 -> 36). Removed every dangling track stub (including a
13 mm antenna on BAT_SENSE and 11 mm on BL_CTRL), one via on BTN_LEFT left
hanging by the stub removal, three AUX_3V3 patch zones that were entirely
isolated dead copper, and one patch zone whose fill was empty. The remaining
patch zones now remove isolated islands on refill. All 36 remaining warnings
are cosmetic silkscreen/text items plus the known Y1 library-footprint note.
DRC: 0 errors, 0 unconnected, 36 warnings. Netlist untouched.
Routing:
- net /RECOVERY: track 97.3 -> 77.0 mm
- net /BAT_SENSE: track 91.0 -> 78.0 mm
- net /UART0_RX: track 46.4 -> 34.0 mm
- net /BL_CTRL: track 63.2 -> 52.2 mm
- net /TFT_DC_CORE: track 41.3 -> 34.2 mm
- net /LCD_D12_FPC: track 19.3 -> 13.3 mm
- net /TFT_SDA_CORE: track 39.3 -> 34.1 mm
- net /LED_A: track 78.4 -> 74.0 mm
- net /LCD_D9_FPC: track 13.4 -> 10.3 mm
- net /LCD_D16_FPC: track 17.1 -> 15.3 mm
- net /BTN_DOWN: track 80.5 -> 79.3 mm
- net /BTN_A: track 101.7 -> 100.5 mm
- net /BTN_RIGHT: track 76.1 -> 74.9 mm
- net /BTN_LEFT: track 94.5 -> 93.3 mm, vias 4 -> 3
- net /TFT_RESET_CORE: track 44.6 -> 43.5 mm
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
Commit message: hw: fix the USB dead-on-arrival findings from the Octavo checklist pass
Self-review against Octavo's OSD335x Schematic Checklist found USB0_VBUS (J16)
fed 2.5 V by the R3/R4 10k/10k divider - below the PHY's 4.4 V session-valid
threshold, so USB device mode and USB boot recovery could never work. The ball
is 5 V-tolerant and nothing else uses the divided net (verified: net members
are C1, R3, R4, J16 only), so R3 becomes 0R and R4 is DNP; C1 stays as a
filter. R1/R2 22R series resistors on USB0 DP/DM are prohibited by the same
checklist (the PHY terminates internally) and become 0R links.

Value/DNP changes only - no copper moved. DRC 0 errors, ERC unchanged,
CPL regenerated (100 placements, R4 now excluded), BOM and spec updated.
Parts:
- R1, R2: value 22R -> 0R
- R3: value 10k -> 0R
- R4: value 10k -> 10k DNP
Changed lines of the file:
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@@
 			)
 		)
-		(property "Value" "10k"
+		(property "Value" "0R"
 			(at 0 1.17 90)
 			(layer "F.Fab")
@@
 			)
 		)
-		(property "Value" "10k"
+		(property "Value" "10k DNP"
 			(at 0 1.17 90)
 			(layer "F.Fab")
@@
 		(sheetname "/")
 		(sheetfile "pokeboy-hw.kicad_sch")
-		(attr smd)
+		(attr smd exclude_from_pos_files dnp)
 		(fp_line
 			(start -0.153641 -0.38)
@@
 			)
 		)
-		(property "Value" "22R"
+		(property "Value" "0R"
 			(at 0 1.17 90)
 			(layer "F.Fab")
@@
 			)
 		)
-		(property "Value" "22R"
+		(property "Value" "0R"
 			(at 0 1.17 90)
 			(layer "F.Fab")
