File: hardware/pokeboy-hw/pokeboy-hw.kicad_sch (KiCad schematic)
At the start: 99 parts, among them J1 USB Micro-B data/power, J2 LiPo 1S + / NTC / -, J3 POWER SWITCH PADS, J4 8 OHM SPEAKER PADS, J5 EA TFT020-23AINN RGB666, J6 UART TEST PADS, J7 RECOVERY SHORT PADS, J8 RESET SHORT PADS, SW1 EVQ-P1905M, SW2 EVQ-P1905M, SW3 EVQ-P1905M, SW4 EVQ-P1905M, SW5 B3AL-1001P, SW6 B3AL-1001P, SW7 EVQ-P2B02B, SW8 EVQ-P2B02B, U1 Core1106, U2 BQ24074RGT, U3 TPS63802DLAR, U4 TPS62162DSG, U5 TPS61165DRV, U6 PAM8302AAD, U7 TPD2EUSB30

Commit message: hw: retarget SoM to Octavo OSD3358-1G-ISM (1 GB DDR3L)
Move the main SoM to OSD3358-1G-ISM: 1 GB DDR3L in a 21x21 mm 256-BGA,
1.27 mm pitch, with integrated PMIC. PocketBeagle is the reference design.

- Add Pokeboy.pretty/OSD335X-BGA-256.kicad_mod, adapted from the
  BeagleBoard.org PocketBeagle design (CC BY 4.0); attribution in
  hardware/pokeboy-hw/THIRD_PARTY_NOTICES.md.
- Update schematic, PCB, Core1106 symbol, and the :6767 preview
  renders/FAB_NOTES for the new part.
- Drop the stale PROTO-A fabrication/gerber/source zips. They describe
  the superseded revision and must not be fabricated.

Status: PROTO-B, DFM HOLD. DRC shows no shorts or spacing violations but
still reports 15 unconnected items (SD_D0-D3/SD_CMD/SD_CD_N to the
R104-R109 pullups, OSD_3V3A, SYS_5V, and GND/AUX_3V3 zone islands).
Gerbers are withheld until DRC is clean. Not releasable for fabrication.
Parts:
- U1: value Core1106 -> OSD3358-1G compute subsystem; footprint Core1106-PCB:Core1106-SMT -> Pokeboy:OSD335X-BGA-256; MPN Core11060408 -> OSD3358-1G-ISM; Notes 30x30 mm SoM; underside components require carrier aperture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 -> 21x21x2 mm direct BGA; 1 GB integrated DDR3L; external micr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
- U6: value PAM8302AAD -> MAX98357AETE+T (PCB canonical); MPN PAM8302AADCR -> MAX98357AETE+T; Notes Single-ended input; differential BTL output -> PCB uses I2S input and differential BTL output; legacy symb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
Other:
- title: Pokeboy Core1106 low-profile carrier -> Pokeboy OSD3358-1G low-profile carrier
Changed lines of the file:
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@@
 	(paper "A0")
 	(title_block
-		(title "Pokeboy Core1106 low-profile carrier")
+		(title "Pokeboy OSD3358-1G low-profile carrier")
 		(date "2026-08-15")
-		(rev "PROTO-A")
+		(rev "PROTO-B DFM HOLD")
 		(company "Pokeboy")
-		(comment 1 "0.8 mm four-layer PCB; Core underside aperture; modelled top envelope ~2.6 mm")
+		(comment 1 "0.8 mm four-layer PCB; 21 mm direct BGA; modelled top envelope 2.0 mm")
 		(comment 2 "EA TFT020-23AINN native RGB666; protected 1S LiPo; Micro-USB data + charge")
 		(comment 3 "Validate panel timing/serial initialization and thermals on first article")
-		(comment 4 "Core1106 variant: Core11060408 (256 MB DDR3L + 8 GB eMMC)")
+		(comment 4 "Compute: OSD3358-1G-ISM (1 GB DDR3L); microSD boot; PCB ball map is canonical")
 	)
 	(symbol
@@
 			)
 		)
-		(property "Value" "Core1106"
+		(property "Value" "OSD3358-1G compute subsystem"
 			(at 226.06 63.5 0)
 			(effects
@@
 			)
 		)
-		(property "Footprint" "Core1106-PCB:Core1106-SMT"
+		(property "Footprint" "Pokeboy:OSD335X-BGA-256"
 			(at 103.632 65.024 0)
 			(effects
@@
 			)
 		)
-		(property "Description" "Core1106"
+		(property "Description" "Logical interface; PCB ball map and PocketBeagle reference are canonical"
 			(at 93.472 61.468 0)
 			(effects
@@
 			)
 		)
-		(property "MPN" "Core11060408"
+		(property "MPN" "OSD3358-1G-ISM"
 			(at 88.9 71.1199 0)
 			(effects
@@
 			)
 		)
-		(property "Notes" "30x30 mm SoM; underside components require carrier aperture; 8 GB eMMC on-module"
+		(property "Notes" "21x21x2 mm direct BGA; 1 GB integrated DDR3L; external microSD boot"
 			(at 88.9 71.1199 0)
 			(effects
@@
 			)
 		)
-		(property "Value" "PAM8302AAD"
+		(property "Value" "MAX98357AETE+T (PCB canonical)"
 			(at 462.28 403.86 0.0000)
 			(effects
@@
 			)
 		)
-		(property "MPN" "PAM8302AADCR"
+		(property "MPN" "MAX98357AETE+T"
 			(at 457.2 400.0499 0)
 			(effects
@@
 			)
 		)
-		(property "Notes" "Single-ended input; differential BTL output"
+		(property "Notes" "PCB uses I2S input and differential BTL output; legacy symbol is logical only"
 			(at 457.2 400.0499 0)
 			(effects

Commit message: hw: reconcile the schematic to the board and clean up the CPL
The schematic did not describe this board. It still held the Luckfox
Core1106 (Rockchip RV1106, 112 numeric pins) as U1 while the board is an
Octavo OSD3358 BGA-256; 17 parts existed only in the PCB; 6 existed only
in the schematic; and ERC therefore only ever covered 99 of 110 parts.

Schematic, matching the sheet's existing style (labels on pins, no wires):

- Replace U1 with an OSD3358_BGA256 symbol whose 132 pins are the ball
  designators the board uses. GENERATED FROM THE LAYOUT - it makes the two
  files agree, it does not verify the ball map against Octavo's datasheet.
- Add the 17 PCB-only parts: Y1, J9, RN7-RN10, R102, R104-R109, C102,
  C103, C105, C106. New symbols for the crystal, an 11-way connector and
  a real MAX98357A (U6 was a PAM8302AAD, 8 pins, MSOP-8).
- Drop the obsolete analog line-in path C17/C18/C19/R24/R25 - the board
  has no CODEC_LINEOUT/LINE_FILT/AMP_IN nets, U6 is I2S.
- Correct C20/C21: schematic had them on AUX_3V3, the board has them on
  SYS_5V beside U6, whose VDD is SYS_5V.
- Remove 45 no-connects left dangling by the U1 swap; snap new placement
  to the 1.27 mm grid.

Board:

- Add R26, the 100k AMP_EN pull-down, at (17.5,36.0). It was schematic-
  only, so the amp enable had no pull-down; it also consumes a dangling
  AMP_EN stub.
- Mark R9/R19 DNP and exclude J2-J8 from pos files. DNP previously lived
  only in the hand-written BOM, so the CPL told the assembler to fit
  parts the BOM says not to fit. CPL drops 109 -> 101 placeable rows.
- Library-qualify all 18 unqualified footprint ids, register
  Connector_Card, and export the crystal footprint to Pokeboy.pretty.

Verification: schematic netlist and PCB connectivity are now identical -
0 nets differing in membership, none present on only one side. DRC 0
errors / 0 unconnected / 80 warnings (was 99). ERC 5, down from 87 once
it began covering all 110 parts.

Two real defects found and NOT fixed, both needing the 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
Parts:
- removed C17, C18, C19: 1u, Capacitor_SMD:C_0402_1005Metric, symbol Device:C
- removed R24: 100R, Resistor_SMD:R_0402_1005Metric, symbol Device:R
- removed R25: 33k, Resistor_SMD:R_0402_1005Metric, symbol Device:R
- removed U1: OSD3358-1G compute subsystem, Pokeboy:OSD335X-BGA-256, symbol Core1106:Core1106
- removed U6: MAX98357AETE+T (PCB canonical), Package_SO:MSOP-8_3x3mm_P0.65mm, symbol Amplifier_Audio:PAM8302AAD
- added C102, C103: 18pF, Capacitor_SMD:C_0402_1005Metric, symbol Device:C
- added C105: 100nF, Capacitor_SMD:C_0402_1005Metric, symbol Device:C
- added C106: 10uF, Capacitor_SMD:C_0805_2012Metric, symbol Device:C
- added J9: 104031-0811, Connector_Card:microSD_HC_Molex_104031-0811, symbol Connector_Generic:Conn_01x11
- added R102: 1M, Resistor_SMD:R_0402_1005Metric, symbol Device:R
- added R104, R105, R106, R107, R108, R109: 10k, Resistor_SMD:R_0402_1005Metric, symbol Device:R
- added RN10, RN7, RN8, RN9: 100k, Resistor_SMD:R_Array_Convex_4x0603, symbol Device:R_Pack04
- added U1: OSD3358-1G-ISM, Pokeboy:OSD335X-BGA-256, symbol Core1106:OSD3358_BGA256
- added U6: MAX98357AETE+T, Package_DFN_QFN:TQFN-16-1EP_3x3mm_P0.5mm_EP1.23x1.23mm, symbol Amplifier_Audio:MAX98357A
- added Y1: 24 MHz, Pokeboy:CRYSTAL_5X3.2MM, symbol Device:Crystal
- R19, R9: now not fitted
Connections:
- net AMP_EN: now also U1.B4 (AMP_EN), U6.4 (SD_MODE)
- net AMP_OUT_N: now also U6.10 (OUTN)
- net AMP_OUT_P: now also U6.9 (OUTP)
- net AUX_3V3: no longer C20.1, C21.1
- net BAT_SENSE: now also U1.A8 (BAT_SENSE)
- net BL_CTRL: now also U1.C3 (BL_CTRL)
- net BTN_A: now also U1.A13 (BTN_A)
- net BTN_B: now also U1.A14 (BTN_B)
- net BTN_DOWN: now also U1.A11 (BTN_DOWN)
- net BTN_LEFT: now also U1.A3 (BTN_LEFT)
- net BTN_RIGHT: now also U1.A4 (BTN_RIGHT)
- net BTN_SELECT: now also U1.B1 (BTN_SELECT)
- net BTN_START: now also U1.B3 (BTN_START)
- net BTN_UP: now also U1.A10 (BTN_UP)
- net CHG_ACTIVE_N: now also U1.C13 (CHG_ACTIVE_N)
- net CHG_PGOOD_N: now also U1.R7 (CHG_PGOOD_N)
- net GND: now also C102.2, C103.2, C105.2, C106.2, J9.10 (Pin_10), J9.6 (Pin_6), RN10.1 (R1.1), RN10.2 (R2.1), RN10.3 (R3.1), RN7.5 (R4.2), RN7.6 (R3.2), RN7.8 (R1.2), RN8.5 (R4.2), RN8.6 (R3.2), RN8.7 (R2.2), RN8.8 (R1.2), RN9.6 (R3.2), RN9.7 (R2.2), RN9.8 (R1.2), U1.D8 (GND), U1.D9 (GND), U1.E10 (GND), U1.E11 (GND), U1.E12 (GND), U1.E5 (GND), U1.E6 (GND), U1.E7 (GND), U1.E8 (GND), U1.E9 (GND), U1.F12 (GND), U1.F5 (GND), U1.G12 (GND), U1.G5 (GND), U1.H12 (GND), U1.H13 (GND), U1.H4 (GND), U1.H5 (GND), U1.J12 (GND), U1.J13 (GND), U1.J4 (GND), U1.J5 (GND), U1.K12 (GND), U1.K5 (GND), U1.L12 (GND), U1.L5 (GND), U1.M10 (GND), U1.M11 (GND), U1.M12 (GND), U1.M5 (GND), U1.M6 (GND), U1.M7 (GND), U1.M8 (GND), U1.M9 (GND), U1.N15 (GND), U1.N8 (GND), U1.N9 (GND), U6.11 (GND), U6.15 (GND), U6.17 (EP), U6.2 (GND), U6.3 (GND)
- net LCD_CLK_CORE: now also U1.F1 (LCD_CLK_CORE)
- net LCD_D0_CORE: now also RN10.8 (R1.2), U1.G3 (LCD_D0_CORE)
- net LCD_D10_CORE: now also RN8.2 (R2.1), U1.K2 (LCD_D10_CORE)
- net LCD_D11_CORE: now also RN8.1 (R1.1), U1.K1 (LCD_D11_CORE)
- net LCD_D12_CORE: now also RN7.4 (R4.1), U1.L3 (LCD_D12_CORE)
- net LCD_D13_CORE: now also RN7.3 (R3.1), U1.L2 (LCD_D13_CORE)
- net LCD_D14_CORE: now also RN7.2 (R2.1), U1.L1 (LCD_D14_CORE)
- net LCD_D15_CORE: now also RN7.1 (R1.1), U1.M3 (LCD_D15_CORE)
- net LCD_D16_CORE: now also U1.P7 (LCD_D16_CORE)
- net LCD_D17_CORE: now also U1.T6 (LCD_D17_CORE)
- net LCD_D1_CORE: now also RN10.7 (R2.2), U1.G2 (LCD_D1_CORE)
- net LCD_D2_CORE: now also RN10.6 (R3.2), U1.G1 (LCD_D2_CORE)
- net LCD_D3_CORE: now also RN10.5 (R4.2), U1.H3 (LCD_D3_CORE)
- net LCD_D4_CORE: now also RN9.4 (R4.1), U1.H2 (LCD_D4_CORE)
- net LCD_D5_CORE: now also RN9.3 (R3.1), U1.H1 (LCD_D5_CORE)
- net LCD_D6_CORE: now also RN9.2 (R2.1), U1.J3 (LCD_D6_CORE)
- net LCD_D7_CORE: now also RN9.1 (R1.1), U1.J2 (LCD_D7_CORE)
- net LCD_D8_CORE: now also RN8.4 (R4.1), U1.J1 (LCD_D8_CORE)
- net LCD_D9_CORE: now also RN8.3 (R3.1), U1.K3 (LCD_D9_CORE)
- net LCD_DE_CORE: now also U1.E1 (LCD_DE_CORE)
- net LCD_HSYNC_CORE: now also U1.F2 (LCD_HSYNC_CORE)
- net LCD_VSYNC_CORE: now also U1.F3 (LCD_VSYNC_CORE)
- net NPOR: now also U1.R11 (NPOR)
- net RECOVERY: now also U1.C1 (RECOVERY)
- net SYS_5V: now also C20.1, C21.1, C106.1, U1.P10 (SYS_5V), U1.R10 (SYS_5V), U1.T10 (SYS_5V), U6.7 (VDD), U6.8 (VDD)
- net TFT_DC_CORE: now also U1.C5 (TFT_DC_CORE)
- net TFT_RESET_CORE: now also U1.C12 (TFT_RESET_CORE)
- net TFT_SCL_CORE: now also U1.C10 (TFT_SCL_CORE)
- net TFT_SDA_CORE: now also U1.C11 (TFT_SDA_CORE)
- net UART0_RX: now also U1.A12 (UART0_RX)
- net UART0_TX: now also U1.B12 (UART0_TX)
- net USB_DM: now also U1.K16 (USB_DM)
- net USB_DP: now also U1.K15 (USB_DP)
- net USB_VBUSDET: now also U1.J16 (USB_VBUSDET)
- new net I2S_BCLK: U1.A1 (I2S_BCLK), U6.16 (BCLK)
- new net I2S_DOUT: U1.B2 (I2S_DOUT), U6.1 (DIN)
- new net I2S_LRCLK: U1.A2 (I2S_LRCLK), U6.14 (LRCLK)
- new net OSD_1V8: U1.F10 (OSD_1V8), U1.G10 (OSD_1V8), U1.H10 (OSD_1V8), U1.H11 (OSD_1V8), U1.J10 (OSD_1V8), U1.J11 (OSD_1V8), U1.K10 (OSD_1V8), U1.L10 (OSD_1V8)
- new net OSD_3V3A: J9.4 (Pin_4), R104.2, R105.2, R106.2, R107.2, R108.2, R109.2, U1.F8 (OSD_3V3A), U1.F9 (OSD_3V3A), U1.G8 (OSD_3V3A), U1.G9 (OSD_3V3A), U1.H7 (OSD_3V3A), U1.H8 (OSD_3V3A), U1.H9 (OSD_3V3A), U1.J7 (OSD_3V3A), U1.J8 (OSD_3V3A), U1.J9 (OSD_3V3A), U1.K8 (OSD_3V3A), U1.K9 (OSD_3V3A), U1.L8 (OSD_3V3A), U1.L9 (OSD_3V3A)
- new net OSD_3V3AUX: U1.F11 (OSD_3V3AUX), U1.G11 (OSD_3V3AUX)
- new net OSD_3V3B: C105.1, RN10.4 (R4.1), RN7.7 (R2.2), RN9.5 (R4.2), U1.F6 (OSD_3V3B), U1.F7 (OSD_3V3B), U1.G6 (OSD_3V3B), U1.G7 (OSD_3V3B)
- new net OSD_OSC_IN: C102.1, R102.1, U1.P16 (OSD_OSC_IN), Y1.2
- new net OSD_OSC_OUT: C103.1, R102.2, U1.N16 (OSD_OSC_OUT), Y1.1
- new net OSD_RTC_1V8: U1.K11 (OSD_RTC_1V8), U1.L11 (OSD_RTC_1V8)
- new net OSD_SYS: U1.K6 (OSD_SYS), U1.K7 (OSD_SYS), U1.L6 (OSD_SYS), U1.L7 (OSD_SYS)
- new net SD_CD_N: J9.9 (Pin_9), R109.1, U1.C14 (SD_CD_N)
- new net SD_CLK: J9.5 (Pin_5), U1.B15 (SD_CLK)
- new net SD_CMD: J9.3 (Pin_3), R108.1, U1.B16 (SD_CMD)
- new net SD_D0: J9.7 (Pin_7), R104.1, U1.A16 (SD_D0)
- new net SD_D1: J9.8 (Pin_8), R105.1, U1.A15 (SD_D1)
- new net SD_D2: J9.1 (Pin_1), R106.1, U1.C16 (SD_D2)
- new net SD_D3: J9.2 (Pin_2), R107.1, U1.C15 (SD_D3)
- no-connect marks 56 -> 16

Commit message: hw: verify U1's ball map against Octavo and tie the balls it requires
The OSD3358 symbol was generated from the layout, so it could only prove the
schematic and the board agreed - not that either was right. Checking it against
Octavo's own PocketBeagle reference design (OSD3358-512M-BSM, identical BGA-256
ball map) confirms every peripheral assignment: LCD, MMC0, I2C0, UART0, MCASP0,
USB0 and OSC0 all land on balls whose documented signal names match. Pin names
in the symbol now come from that library, so the sheet shows the datasheet
signal beside the net and any future divergence is visible.

The same check found balls the reference ties that this board left floating:

- N10/N11 PMIC_POWER_EN <-> PMIC_PWR_EN. This gates the PMIC's enable, so as it
  stood the SiP would not have powered up at all.
- N4/N5 PMIC_LDO_PGOOD <-> RTC_PWRONRSTN.
- N12/P11 PMIC_PGOOD -> PWRONRSTN, which releases reset.
- A7/B7 SYS_ADC_1P8V -> VREFP and A9/B9 AGND_ADC -> VREFN. AIN0 is in use for
  BAT_SENSE, and without a reference pair that reading is meaningless.

All five are adjacent-ball ties inside the 1.27 mm field, routed on F.Cu.

The two stranded Core1106 rails are also retired:

- CORE_3V3 fed R12/R13/R18/R32 from nothing. Its pull-ups all bias nets in the
  VDDSHV I/O domain, so it is merged onto OSD_3V3A, which supplies that domain.
  SD_CLK walls off F.Cu at x=50.772 and the SD fanout fills In1 and In2 in the
  gap, so no new via fits; both sides already own a through via and B.Cu between
  them is clear, so the join is one bottom-layer track and no new via.
- The In1 spine and F.Cu stub that carried CORE_3V3 west to the old module's
  landing pads are removed - R12/R13/R18 reach the net over In2 and R32 on F.Cu.
- CORE_1V8 reached only TP1. All eight SYS_VDD_1P8V balls sit in the interior of
  the field ringed by DGND, and Octavo's own PocketBeagle leaves VDD_1V8 with no
  external connection either, so the rail cannot be brought out. TP1 is removed
  rather than left wired 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
Parts:
- removed TP1: CORE 1V8 TEST, TestPoint:TestPoint_Pad_D1.0mm, symbol Connector:TestPoint
Connections:
- net CORE_3V3 is gone; now on net OSD_3V3A: R12.1, R13.1, R18.1, R32.1
- net GND: now also J9.11 (Pin_11)
- new net ADC_VREFN: U1.A9 (AGND_ADC), U1.B9 (VREFN)
- new net ADC_VREFP: U1.A7 (SYS_ADC_1P8V), U1.B7 (VREFP)
- new net PMIC_PGOOD: U1.N12 (PMIC_PGOOD), U1.P11 (PWRONRSTN)
- new net PMIC_PWR_EN: U1.N10 (PMIC_POWER_EN), U1.N11 (PMIC_PWR_EN)
- new net RTC_PWRONRSTN: U1.N4 (PMIC_LDO_PGOOD), U1.N5 (RTC_PWRONRSTN)

Commit message: hw: fix the USB dead-on-arrival findings from the Octavo checklist pass
Self-review against Octavo's OSD335x Schematic Checklist found USB0_VBUS (J16)
fed 2.5 V by the R3/R4 10k/10k divider - below the PHY's 4.4 V session-valid
threshold, so USB device mode and USB boot recovery could never work. The ball
is 5 V-tolerant and nothing else uses the divided net (verified: net members
are C1, R3, R4, J16 only), so R3 becomes 0R and R4 is DNP; C1 stays as a
filter. R1/R2 22R series resistors on USB0 DP/DM are prohibited by the same
checklist (the PHY terminates internally) and become 0R links.

Value/DNP changes only - no copper moved. DRC 0 errors, ERC unchanged,
CPL regenerated (100 placements, R4 now excluded), BOM and spec updated.
Parts:
- R1, R2: value 22R -> 0R
- R3: value 10k -> 0R
- R4: now not fitted
Changed lines of the file:
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@@
 			)
 		)
-		(property "Value" "22R"
+		(property "Value" "0R"
 			(at 510.54 30.48 90)
 			(effects
@@
 			)
 		)
-		(property "Value" "22R"
+		(property "Value" "0R"
 			(at 510.54 39.37 90)
 			(effects
@@
 			)
 		)
-		(property "Value" "10k"
+		(property "Value" "0R"
 			(at 469.9 54.61 90)
 			(effects
@@
 		(in_bom yes)
 		(on_board yes)
-		(dnp no)
+		(dnp yes)
 		(fields_autoplaced no)
 		(property "Reference" "R4"

Commit message: hw: close the Octavo checklist copper items
- SYS_VOUT bulk (PD4, was mandatory-and-missing): C107-C109, three 22 uF 0402
  (same GRM155R61A226ME11D as C7/C8, 66 uF nominal to survive DC-bias derating)
  placed below U1 at y=9.7, fed by a 0.3 mm F.Cu trunk down the col-6/7 ball
  gap from the existing SYS_VOUT interlink; GND pads land in the F.Cu pour.
- VIN_BAT (P8/R8/T8) strapped to PMIC_BAT_SENSE (N7) as new net /VIN_BAT;
  VIN_USB (P9/R9/T9) tied to GND via the N9 ball - Table 13 Use Case 4.
- EEPROM_WP (M2) tied to GND.
- 12 GND stitching vias added beside DGND balls under U1 (was 2 in the whole
  field), each collision-checked on all four layers; drill 227 -> 239 hits.
- U1's schematic symbol gains the 8 previously-floating pins; 3 cap symbols
  added; netlist and board verified identical net for net.

DRC 0 errors / 0 unconnected / 37 warnings (one new cosmetic silk-over-copper
from the cap refs). ERC 0 errors / 4 baseline warnings. Fab outputs, CPL (103
placements), BOM, renders, copper SVGs, STEP, schematic PDF regenerated.

Software note carried in HANDOVER: disable the TPS65217 charger (external
BQ24074 charges the cell) and cap the sustained OPP per the thermal plan.
Parts:
- added C107, C108, C109: 22u/10V, Capacitor_SMD:C_0402_1005Metric, symbol Device:C
Connections:
- net GND: now also U1.M2 (EEPROM_WP), U1.P9 (VIN_USB), U1.R9 (VIN_USB), U1.T9 (VIN_USB), C107.2, C108.2, C109.2
- net OSD_SYS: now also C107.1, C108.1, C109.1
- new net VIN_BAT: U1.N7 (PMIC_BAT_SENSE), U1.P8 (VIN_BAT), U1.R8 (VIN_BAT), U1.T8 (VIN_BAT)

Commit message: PROTO-B1: fix all design-review findings, DRC/ERC clean
Design review (2026-08-18) found the PROTO-B package unbuildable. All
findings fixed and verified; full record in
hardware/manufacturing/pcbway/OPEN_DESIGN_ISSUES.md.

- U7: TPD2EUSB30DRTR was on a SOT-23-3 land; now Texas_DRT-3, pocket
  re-routed (D+ to In1 below pad 1, D- via In1 spine)
- USB: R1/R2 0R jumpers removed; USB_DP/USB_DM one continuous net per
  leg J1 -> U7 -> U1; stale stubs and redundant vias deleted
- J5: exclude_from_pos_files removed so the WF030-39S FFC connector is
  actually placed (CPL 102 placements); BOM row split connector/panel;
  pin 35 IM3 strap GND -> AUX_3V3 per EA TFT020-23AI RGB mode
- BQ24074: EN1 strap AUX_3V3 -> VBUS; batteryless USB plug-in now
  starts in USB500 instead of deadlocking at USB100
- SYS_VOUT bulk: C107-C109 to 22uF/10V 0805 (GRM21BR61A226ME44L),
  respaced 2.2mm, rail extended (Octavo ~50uF requirement)
- BOM: nonexistent GRM155 22uF MPNs corrected to real GRM158 parts;
  J3/display/switch off-board rows added; MSL 4 stated in fab docs
- RECOVERY net renamed JTAG_TDI (J7 is a TDI test pad; SYSBOOT already
  falls through to USB0 for recovery)
- Y1 resynced from Pokeboy.pretty; silk cleaned to zero warnings;
  mask colour Black in stackup; rev PROTO-B1 on silk and title block

DRC 0 errors / 0 warnings / 0 unconnected; ERC 0 errors.
Full fab regen: gerbers, drills+maps, IPC-D-356, CPL, LAYERS.txt,
PROTO-B1 zips (old PROTO-B zips removed).
Parts:
- removed R1, R2: 0R, Resistor_SMD:R_0402_1005Metric, symbol Device:R
- C107, C108, C109: footprint Capacitor_SMD:C_0402_1005Metric -> Capacitor_SMD:C_0805_2012Metric
- J5: value EA TFT020-23AINN RGB666 -> EA WF030-39S
- U7: footprint Package_TO_SOT_SMD:SOT-23-3 -> Package_TO_SOT_SMD:Texas_DRT-3
Connections:
- net USB_DM_CONN is gone; now on net USB_DM: J1.2 (D-), U7.2 (D-)
- net USB_DP_CONN is gone; now on net USB_DP: J1.3 (D+), U7.1 (D+)
- net AUX_3V3: now also J5.35 (Pin_35); no longer U2.6 (EN1)
- net GND: no longer J5.35 (Pin_35)
- net VBUS: now also U2.6 (EN1)
- net RECOVERY renamed JTAG_TDI
Changed lines of the file:
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@@
 		(title "Pokeboy OSD3358-1G low-profile carrier")
 		(date "2026-08-15")
-		(rev "PROTO-B DFM HOLD")
+		(rev "PROTO-B1")
 		(company "Pokeboy")
 		(comment 1 "0.8 mm four-layer PCB; 21 mm direct BGA; modelled top envelope 2.0 mm")
@@
 			)
 		)
-		(property "Footprint" "Package_TO_SOT_SMD:SOT-23-3"
+		(property "Footprint" "Package_TO_SOT_SMD:Texas_DRT-3"
 			(at 469.9 35.56 0)
 			(effects
@@
 	(symbol
 		(lib_id "Device:R")
-		(at 510.54 30.48 0)
-		(unit 1)
-		(exclude_from_sim no)
-		(in_bom yes)
-		(on_board yes)
-		(dnp no)
-		(fields_autoplaced no)
-		(property "Reference" "R1"
-			(at 512.572 30.48 90)
-			(effects
-				(font
-					(size 1.27 1.27)
-				)
-				(justify left)
-			)
-		)
-		(property "Value" "0R"
-			(at 510.54 30.48 90)
-			(effects
-				(font
-					(size 1.27 1.27)
-				)
-				(justify left)
-			)
-		)
-		(property "Footprint" "Resistor_SMD:R_0402_1005Metric"
-			(at 510.54 30.48 0)
-			(effects
-				(font
-					(size 1.27 1.27)
-				)
-				(hide yes)
-			)
-		)
-		(pin "1"
-		)
-		(pin "2"
-		)
-		(instances
-			(project "pokeboy-hw"
-				(path "/61fdeb8d-5442-41ae-99a5-d057c2041497"
-					(reference "R1")
-					(unit 1)
-				)
-			)
-		)
-	)
-	(symbol
-		(lib_id "Device:R")
-		(at 510.54 39.37 0)
-		(unit 1)
-		(exclude_from_sim no)
-		(in_bom yes)
-		(on_board yes)
-		(dnp no)
-		(fields_autoplaced no)
-		(property "Reference" "R2"
-			(at 512.572 39.37 90)
-			(effects
-				(font
-					(size 1.27 1.27)
-				)
-				(justify left)
-			)
-		)
-		(property "Value" "0R"
-			(at 510.54 39.37 90)
-			(effects
-				(font
-					(size 1.27 1.27)
-				)
-				(justify left)
-			)
-		)
-		(property "Footprint" "Resistor_SMD:R_0402_1005Metric"
-			(at 510.54 39.37 0)
-			(effects
-				(font
-					(size 1.27 1.27)
-				)
-				(hide yes)
-			)
-		)
-		(pin "1"
-		)
-		(pin "2"
-		)
-		(instances
-			(project "pokeboy-hw"
-				(path "/61fdeb8d-5442-41ae-99a5-d057c2041497"
-					(reference "R2")
-					(unit 1)
-				)
-			)
-		)
-	)
-	(symbol
-		(lib_id "Device:R")
 		(at 469.9 54.61 0)
 		(unit 1)
@@
 			)
 		)
-		(property "Value" "EA TFT020-23AINN RGB666"
+		(property "Value" "EA WF030-39S"
 			(at 720.09 144.78 0.0000)
 			(effects
@@
 		)
 	)
-	(label "USB_DM_CONN"
+	(label "USB_DM"
 		(at 433.07 38.1 0.0000)
 		(effects
@@
 		)
 	)
-	(label "USB_DP_CONN"
+	(label "USB_DP"
 		(at 433.07 35.56 0.0000)
 		(effects
@@
 		)
 	)
-	(label "USB_DP_CONN"
+	(label "USB_DP"
 		(at 459.74 35.56 0.0000)
 		(effects
@@
 		)
 	)
-	(label "USB_DM_CONN"
+	(label "USB_DM"
 		(at 480.06 35.56 0.0000)
 		(effects
@@
 		)
 	)
-	(label "USB_DP_CONN"
-		(at 510.54 26.67 0.0000)
-		(effects
-			(font
-				(size 1 1)
-			)
-			(justify left bottom)
-		)
-	)
-	(label "USB_DP"
-		(at 510.54 34.29 0.0000)
-		(effects
-			(font
-				(size 1 1)
-			)
-			(justify left bottom)
-		)
-	)
-	(label "USB_DM_CONN"
-		(at 510.54 35.56 0.0000)
-		(effects
-			(font
-				(size 1 1)
-			)
-			(justify left bottom)
-		)
-	)
-	(label "USB_DM"
-		(at 510.54 43.18 0.0000)
-		(effects
-			(font
-				(size 1 1)
-			)
-			(justify left bottom)
-		)
-	)
 	(label "VBUS"
 		(at 469.9 50.8 0.0000)
@@
 		)
 	)
-	(label "AUX_3V3"
+	(label "VBUS"
 		(at 447.04 105.41 0.0000)
 		(effects
@@
 		)
 	)
-	(label "GND"
+	(label "AUX_3V3"
 		(at 715.01 233.68 0.0000)
 		(effects
@@
 		)
 	)
-	(label "RECOVERY"
+	(label "JTAG_TDI"
 		(at 679.45 469.9 0.0000)
 		(effects
@@
 		)
 	)
-	(label "RECOVERY"
+	(label "JTAG_TDI"
 		(at 457.2 621.03 0.0000)
 		(effects
@@
 			)
 		)
-		(property "Footprint" "Capacitor_SMD:C_0402_1005Metric"
+		(property "Footprint" "Capacitor_SMD:C_0805_2012Metric"
 			(at 594.36 175.26 0)
 			(effects
@@
 			)
 		)
-		(property "Footprint" "Capacitor_SMD:C_0402_1005Metric"
+		(property "Footprint" "Capacitor_SMD:C_0805_2012Metric"
 			(at 612.14 175.26 0)
 			(effects
@@
 			)
 		)
-		(property "Footprint" "Capacitor_SMD:C_0402_1005Metric"
+		(property "Footprint" "Capacitor_SMD:C_0805_2012Metric"
 			(at 629.92 175.26 0)
 			(effects
